File: hs-probe.sch (KiCad schematic (older format))
At the start: 45 parts, among them J1 USB_C_Receptacle_USB2.0, U1 STM32F723IEKx, U2 DSC6003HI2A-012.0000T, U3 MIC5259, U4 NUF8401MNT4G, U5 STDC14, U6 SOICbite_SWD, U7 MIC5259

Commit message: Fix errors
Connections:
- net LED1: now also U1.B14 (PC10); no longer U1.A15 (PA13)
- net OSC: now also U1.G1 (PH0); no longer U1.M7 (PG1)
- net P_SWDIO: now also U1.A15 (PA13); no longer U1.A13 (PA15)
Other:
- moved on the sheet: C3, U2
Changed lines of the file:
@@
 L Oscillator:ASDMB-xxxMHz U2
 U 1 1 5E866432
-P 3750 7150
-F 0 "U2" H 3306 7196 50  0000 R CNN
-F 1 "DSC6003HI2A-012.0000T" H 3306 7105 50  0000 R CNN
-F 2 "crystals:Oscillator_SMD_Abracon_ASCO-4Pin_1.6x1.2mm" H 3750 7150 50  0001 C CNN
-F 3 "http://ww1.microchip.com/downloads/en/DeviceDoc/DSC60XX-Ultra-Small-Ultra-Low-Power-MEMS-Oscillator-DS20005625C.pdf" H 4050 7600 50  0001 C CNN
-	1    3750 7150
-	1    0    0    -1
-$EndComp
-Wire Wire Line
-	5550 7150 4150 7150
+P 3750 5350
+F 0 "U2" H 3306 5396 50  0000 R CNN
+F 1 "DSC6003HI2A-012.0000T" H 3306 5305 50  0000 R CNN
+F 2 "crystals:Oscillator_SMD_Abracon_ASCO-4Pin_1.6x1.2mm" H 3750 5350 50  0001 C CNN
+F 3 "http://ww1.microchip.com/downloads/en/DeviceDoc/DSC60XX-Ultra-Small-Ultra-Low-Power-MEMS-Oscillator-DS20005625C.pdf" H 4050 5800 50  0001 C CNN
+	1    3750 5350
+	1    0    0    -1
+$EndComp
+Wire Wire Line
+	5550 5350 4150 5350
 $Comp
 L power:+3.3V #PWR01
 U 1 1 5E872EDB
-P 3850 6850
-F 0 "#PWR01" H 3850 6700 50  0001 C CNN
-F 1 "+3.3V" H 3865 7023 50  0000 C CNN
-F 2 "" H 3850 6850 50  0001 C CNN
-F 3 "" H 3850 6850 50  0001 C CNN
-	1    3850 6850
+P 3850 5050
+F 0 "#PWR01" H 3850 4900 50  0001 C CNN
+F 1 "+3.3V" H 3865 5223 50  0000 C CNN
+F 2 "" H 3850 5050 50  0001 C CNN
+F 3 "" H 3850 5050 50  0001 C CNN
+	1    3850 5050
 	1    0    0    -1
 $EndComp
@@
 L power:GND #PWR02
 U 1 1 5E875314
-P 3850 7450
-F 0 "#PWR02" H 3850 7200 50  0001 C CNN
-F 1 "GND" H 3855 7277 50  0001 C CNN
-F 2 "" H 3850 7450 50  0001 C CNN
-F 3 "" H 3850 7450 50  0001 C CNN
-	1    3850 7450
-	1    0    0    -1
-$EndComp
-Text Label 4700 7150 0    50   ~ 0
+P 3850 5650
+F 0 "#PWR02" H 3850 5400 50  0001 C CNN
+F 1 "GND" H 3855 5477 50  0001 C CNN
+F 2 "" H 3850 5650 50  0001 C CNN
+F 3 "" H 3850 5650 50  0001 C CNN
+	1    3850 5650
+	1    0    0    -1
+$EndComp
+Text Label 4700 5350 0    50   ~ 0
 OSC
 $Comp
@@
 L Device:C_Small C3
 U 1 1 5E8D1C1D
-P 4650 1850
-F 0 "C3" V 4421 1850 50  0000 C CNN
-F 1 "0.1u" V 4512 1850 50  0000 C CNN
-F 2 "passive:C_0402" H 4650 1850 50  0001 C CNN
-F 3 "~" H 4650 1850 50  0001 C CNN
-	1    4650 1850
-	0    1    1    0
+P 4750 1600
+F 0 "C3" V 4521 1600 50  0000 C CNN
+F 1 "0.1u" V 4612 1600 50  0000 C CNN
+F 2 "passive:C_0402" H 4750 1600 50  0001 C CNN
+F 3 "~" H 4750 1600 50  0001 C CNN
+	1    4750 1600
+	-1   0    0    1
 $EndComp
 $Comp
 L power:GND #PWR09
 U 1 1 5E8D2877
-P 4550 1850
-F 0 "#PWR09" H 4550 1600 50  0001 C CNN
-F 1 "GND" H 4555 1677 50  0001 C CNN
-F 2 "" H 4550 1850 50  0001 C CNN
-F 3 "" H 4550 1850 50  0001 C CNN
-	1    4550 1850
-	0    1    1    0
+P 4750 1500
+F 0 "#PWR09" H 4750 1250 50  0001 C CNN
+F 1 "GND" H 4755 1327 50  0001 C CNN
+F 2 "" H 4750 1500 50  0001 C CNN
+F 3 "" H 4750 1500 50  0001 C CNN
+	1    4750 1500
+	-1   0    0    1
 $EndComp
 Wire Wire Line
@@
 Wire Wire Line
 	5500 2650 5550 2650
-NoConn ~ 3350 7150
+NoConn ~ 3350 5350
 $Comp
 L Device:R_Small R3
@@
 U 1 1 5E9583AD
 P 4650 2150
-F 0 "R1" V 4454 2150 50  0000 C CNN
-F 1 "5.1k" V 4545 2150 50  0000 C CNN
+F 0 "R1" V 4550 2150 50  0000 C CNN
+F 1 "5.1k" V 4750 2150 50  0000 C CNN
 F 2 "passive:R_0402" H 4650 2150 50  0001 C CNN
 F 3 "~" H 4650 2150 50  0001 C CNN
@@
 L power:GND #PWR017
 U 1 1 5E966B7B
-P 5550 1950
-F 0 "#PWR017" H 5550 1700 50  0001 C CNN
-F 1 "GND" H 5555 1777 50  0001 C CNN
-F 2 "" H 5550 1950 50  0001 C CNN
-F 3 "" H 5550 1950 50  0001 C CNN
-	1    5550 1950
+P 4550 1950
+F 0 "#PWR017" H 4550 1700 50  0001 C CNN
+F 1 "GND" H 4555 1777 50  0001 C CNN
+F 2 "" H 4550 1950 50  0001 C CNN
+F 3 "" H 4550 1950 50  0001 C CNN
+	1    4550 1950
 	0    1    1    0
 $EndComp
@@
 Wire Wire Line
 	11150 6200 11250 6200
-Text Label 10550 3050 0    50   ~ 0
+Text Label 10550 6150 0    50   ~ 0
 LED1
 Text Label 10550 2950 0    50   ~ 0
 LED2
-Text Label 10550 3250 0    50   ~ 0
+Text Label 10550 3050 0    50   ~ 0
 P_SWDIO
 Text Label 10550 3150 0    50   ~ 0
@@
 	10550 3150 10450 3150
 Wire Wire Line
-	10450 3250 10550 3250
+	10450 3050 10550 3050
 Text Label 11750 3350 2    50   ~ 0
 P_SWDIO
@@
 LED3
 Wire Wire Line
-	10550 3050 10450 3050
+	10550 6150 10450 6150
 Wire Wire Line
 	10450 2950 10550 2950
@@
 Wire Wire Line
 	12050 6000 12100 6000
+Wire Wire Line
+	4750 1850 4750 1700
+Wire Wire Line
+	4550 1950 5550 1950
 $EndSCHEMATC

Commit message: Added USB Mux to start with FS and then switch to HS
Parts:
- removed D2: ESD7002WTT1G, sot:SOT-323, symbol Device:D_Zener_x2_ACom_KKA
- added C28: 0.1u, passive:C_0402, symbol Device:C_Small
- added R101, R102, R8: 5.1k, passive:R_0402, symbol Device:R_Small
- added U8: USB3740B-AI9, Package_DFN_QFN:UQFN-10_1.6x2.1mm_P0.5mm, symbol Interface_USB:USB3740B-AI9
Connections:
- net +3V3: now also C28.1, U8.5 (VDD); no longer U5.2 (V_PROBE)
- net D_N: now also U8.9 (DM); no longer U1.R14 (PB14)
- net D_P: now also U8.10 (DP); no longer U1.R15 (PB15)
- net GND: now also C28.2, R101.2, R8.2, U8.3 (OE_N), U8.8 (GND)
- net LED2: now also U1.A5 (PB8); no longer U1.B15 (PA12)
- net LED3: now also U1.A4 (PE0); no longer U1.C15 (PA11)
- net T_VCC: now also R102.1; no longer C27.1, U7.4 (VOUT)
- net USB_SEL: now reaches U1.R12 (PB10)
- net USB_SEL: now also R8.1, U8.4 (S)
- net T_VCC_MEAS: now reaches U1.R2 (PA3)
- net T_VCC_MEAS: now also R101.1, R102.2
- new net D_FS_N: U1.C15 (PA11), U8.1 (DM_1)
- new net D_FS_P: U1.B15 (PA12), U8.2 (DP_1)
- new net D_HS_N: U1.R14 (PB14), U8.7 (DM_2)
- new net D_HS_P: U1.R15 (PB15), U8.6 (DP_2)
- new net T_VCC_PWR: C27.1, U5.2 (V_PROBE), U7.4 (VOUT)
Other:
- moved on the sheet: C1, C10, C11, C12, C13, C14, C15, C16, C17, C18, C19, C2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
