File: base.kicad_pcb (KiCad board)
At the start: 4 copper layers, 40 x 14 mm, 55 parts, among them J1 USB_C_Receptacle_USB2.0, J2 Castellated Vias, J3 Castellated Vias, J4 Castellated Vias, J5 tag-connect-swd, U1 hs-probe-stm32, U2 12 MHz, U3 MIC5353, U4 NUF8401MNT4G, U5 STDC14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

Commit message: inital commit
Parts:
- U1: value hs-probe-stm32 -> base-stm32
